Commit message: Update package to add TCP controller for 3f gripper

File: robotiq_3f_gripper_visualization/cfg/robotiq-3f-gripper_articulated_macro.xacro (robot description, xacro)
@@ -43,5 +43,5 @@
 			<axis xyz="0 1 0"/>
 			<origin xyz="-0.0455 0.0214 0.036" rpy="0 3.1416 -1.57"/>
-			<limit lower="-0.1784" upper="0.192" effort="100" velocity="100"/>
+			<limit lower="-0.2" upper="0.192" effort="100" velocity="100"/>
 		</joint>
 		<joint name="${prefix}palm_finger_2_joint" type="revolute">
@@ -50,5 +50,5 @@
 			<axis xyz="0 1 0"/>
 			<origin xyz="-0.0455 0.0214 -0.036" rpy="0 3.1416 -1.57"/>
-			<limit lower="-0.192" upper="0.1784" effort="100" velocity="100"/>
+			<limit lower="-0.192" upper="0.2" effort="100" velocity="100"/>
 		</joint>
 		<joint name="${prefix}palm_finger_middle_joint" type="fixed">
@@ -64,4 +64,13 @@
 		</joint>
 		<!-- end of joint list -->
+		<transmission name="trans_${prefix}palm_finger_1_joint">
+            <type>transmission_interface/SimpleTransmission</type>
+            <joint name="${prefix}palm_finger_1_joint">
+                <hardwareInterface>hardware_interface/PositionJointInterface</hardwareInterface>
+            </joint>
+            <actuator name="${prefix}palm_finger_1_motor">
+                <mechanicalReduction>1</mechanicalReduction>
+            </actuator>
+        </transmission>
 	</xacro:macro>
 </robot>

File: robotiq_3f_gripper_visualization/cfg/robotiq-3f-gripper_finger_articulated_macro.xacro (robot description, xacro)
@@ -125,4 +125,13 @@
 		</joint>
 		<!-- end of joint list -->
+		<transmission name="trans_${prefix}joint_1">
+            <type>transmission_interface/SimpleTransmission</type>
+            <joint name="${prefix}joint_1">
+                <hardwareInterface>hardware_interface/PositionJointInterface</hardwareInterface>
+            </joint>
+            <actuator name="${prefix}joint_1_motor">
+                <mechanicalReduction>1</mechanicalReduction>
+            </actuator>
+        </transmission>
 	</xacro:macro>
 </robot>
